File: orp_adc_iso_hw/orp_adc_iso.brd (EAGLE design)
At the start: 39.4 x 56.8 mm, 25 parts, among them IC1 AD8603AUJZ-REEL7, IC2 LM385MX-2.5_NOPB, IC3 ADS1115IDGSR, IC4 ADUM1250ARZ, J1 RF1-01B-D-00-75

Commit message: used op amp in bigger IC package
Parts:
- removed IC1: AD8603AUJZ-REEL7, AD8603AUJZ-REEL7:SOT95P280X100-5N
- added U$1: LMC6482AIMX/NOPB, other:SO8
- moved J1 6.35 mm to (23.5, 7.62)
- moved C1 4.26 mm to (17.8, 15.7)
Connections:
- new net N$4: U$1.6, U$1.7
- net GND_ISO: now also U$1.4; no longer IC1.2
- net N$2: now also U$1.3; no longer IC1.3
- net N$3: now also U$1.1, U$1.2; no longer IC1.1, IC1.4
- net VCC5V_ISO: now also U$1.8; no longer IC1.5
- net VREF2.5V: now also U$1.5
Routing:
- net N$3: track 30.3 -> 70.7 mm, vias 0 -> 1
- net VREF2.5V: track 49.0 -> 64.7 mm, vias 2 -> 4
- net GND_ISO: track 86.1 -> 70.8 mm, vias 8 -> 11
- net N$4: track 0.00 -> 4.59 mm
- net VCC5V_ISO: track 78.3 -> 79.7 mm
- net N$2: track 4.31 -> 5.66 mm
Other:
- board text added: "3V3"
- board text added: "5V"
- board text added: "GND"
- board text added: "SCL"
- board text added: "SDA"
