File: orp_adc_iso_hw/orp_adc_iso.brd (EAGLE design)
At the start: 39.3 x 62.8 mm, 27 parts, among them IC2 LM385MX-2.5_NOPB, IC3 ADS1115IDGSR, IC4 ADUM1250ARZ, J1 RF1-01B-D-00-75

Commit message: minor movements on pcb
Parts:
- moved C12 1.25 mm to (13.1, 40.0), turned to 90 degrees
- moved C13 0.33 mm to (13.0, 51.4)
Routing:
- net VREF2.5V: track 64.8 -> 67.9 mm, vias 4 -> 3
- net VCC5V_ISO: track 80.7 -> 79.2 mm
Changed lines of the file:
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@@
 <setting verticaltext="up"/>
 </settings>
-<grid distance="1" unitdist="mm" unit="mm" style="dots" multiple="1" display="yes" altdistance="0.01" altunitdist="mm" altunit="mm"/>
+<grid distance="1" unitdist="mm" unit="mm" style="dots" multiple="1" display="yes" altdistance="0.079375" altunitdist="mm" altunit="mm"/>
 <layers>
 <layer number="1" name="Top" color="4" fill="1" visible="yes" active="yes"/>
@@
 <layer number="14" name="Route14" color="1" fill="6" visible="no" active="no"/>
 <layer number="15" name="Route15" color="4" fill="6" visible="no" active="no"/>
-<layer number="16" name="Bottom" color="1" fill="1" visible="no" active="yes"/>
+<layer number="16" name="Bottom" color="1" fill="1" visible="yes" active="yes"/>
 <layer number="17" name="Pads" color="2" fill="1" visible="yes" active="yes"/>
 <layer number="18" name="Vias" color="2" fill="1" visible="yes" active="yes"/>
 <layer number="19" name="Unrouted" color="6" fill="1" visible="yes" active="yes"/>
 <layer number="20" name="Dimension" color="15" fill="1" visible="yes" active="yes"/>
-<layer number="21" name="tPlace" color="7" fill="1" visible="yes" active="yes"/>
+<layer number="21" name="tPlace" color="7" fill="1" visible="no" active="yes"/>
 <layer number="22" name="bPlace" color="7" fill="1" visible="no" active="yes"/>
-<layer number="23" name="tOrigins" color="15" fill="1" visible="yes" active="yes"/>
+<layer number="23" name="tOrigins" color="15" fill="1" visible="no" active="yes"/>
 <layer number="24" name="bOrigins" color="15" fill="1" visible="no" active="yes"/>
 <layer number="25" name="tNames" color="7" fill="1" visible="no" active="yes"/>
@@
 <layer number="49" name="Reference" color="7" fill="1" visible="no" active="yes"/>
 <layer number="50" name="dxf" color="7" fill="1" visible="no" active="no"/>
-<layer number="51" name="tDocu" color="7" fill="1" visible="yes" active="yes"/>
+<layer number="51" name="tDocu" color="7" fill="1" visible="no" active="yes"/>
 <layer number="52" name="bDocu" color="7" fill="1" visible="no" active="yes"/>
 <layer number="53" name="tGND_GNDA" color="7" fill="9" visible="no" active="no"/>
@@
 <element name="U$1" library="other" package="SO8" value="LMC6482AIMX/NOPB" x="20.96" y="15.875" smashed="yes"/>
 <element name="C11" library="rcl" package="SMC_C" value="100 uF" x="8.26" y="26.035" smashed="yes" rot="R270"/>
-<element name="C12" library="rcl" package="SMC_C" value="100 uF" x="13.045" y="38.705" smashed="yes" rot="R270"/>
-<element name="C13" library="rcl" package="SMC_C" value="100 uF" x="12.705" y="51.435" smashed="yes" rot="R270"/>
+<element name="C12" library="rcl" package="SMC_C" value="100 uF" x="13.069375" y="39.955625" smashed="yes" rot="R90"/>
+<element name="C13" library="rcl" package="SMC_C" value="100 uF" x="13.0225" y="51.355625" smashed="yes" rot="R270"/>
 <element name="C7" library="rcl" package="C0603" value="100 nF" x="26.065625" y="25.301875" smashed="yes" rot="R270"/>
 <element name="C9" library="rcl" package="C0603" value="100 nF" x="21.64" y="21.095625" smashed="yes" rot="R180"/>
@@
 <contactref element="IC3" pad="5"/>
 <wire x1="10.9025" y1="30.32125" x2="8.26" y2="30.32125" width="0.4064" layer="1"/>
-<wire x1="8.26" y1="30.32125" x2="8.26" y2="30.559375" width="0.4064" layer="1"/>
 <wire x1="24.61125" y1="26.19375" x2="24.5" y2="26.305" width="0.254" layer="1"/>
 <wire x1="24.5" y1="26.305" x2="24.5" y2="27.01" width="0.254" layer="1"/>
-<via x="8.26" y="30.559375" extent="1-16" drill="0.6"/>
-<wire x1="8.26" y1="30.559375" x2="8.26" y2="30.32125" width="0.4064" layer="16"/>
+<via x="8.26" y="30.32125" extent="1-16" drill="0.6"/>
 <wire x1="8.26" y1="30.32125" x2="27.945" y2="30.32125" width="0.4064" layer="16"/>
-<via x="27.945" y="30.32125" extent="1-16" drill="0.6"/>
-<wire x1="27.945" y1="30.32125" x2="27.945" y2="26.19375" width="0.4064" layer="1"/>
-<wire x1="27.945" y1="26.19375" x2="26.04" y2="26.19375" width="0.254" layer="1"/>
+<wire x1="27.945" y1="26.19375" x2="26.04" y2="26.19375" width="0.4064" layer="1"/>
 <wire x1="26.04" y1="26.19375" x2="24.61125" y2="26.19375" width="0.254" layer="1"/>
-<wire x1="27.945" y1="22.38375" x2="27.945" y2="7.9375" width="0.4064" layer="1"/>
+<wire x1="27.945" y1="26.225" x2="27.945" y2="7.9375" width="0.4064" layer="1"/>
 <wire x1="27.945" y1="7.9375" x2="27.6275" y2="7.62" width="0.4064" layer="1"/>
 <wire x1="27.6275" y1="7.62" x2="24.135" y2="7.62" width="0.4064" layer="1"/>
 <contactref element="U$1" pad="5"/>
-<wire x1="27.945" y1="22.38375" x2="27.945" y2="26.19375" width="0.4064" layer="1"/>
+<wire x1="27.945" y1="26.225" x2="27.945" y2="26.19375" width="0.4064" layer="1"/>
 <wire x1="22.865" y1="18.475" x2="22.865" y2="21.095625" width="0.4064" layer="1"/>
 <via x="22.865" y="22.38375" extent="1-16" drill="0.6"/>
 <wire x1="22.865" y1="21.095625" x2="22.865" y2="22.38375" width="0.4064" layer="1"/>
-<wire x1="22.865" y1="22.38375" x2="27.945" y2="22.38375" width="0.4064" layer="16"/>
-<via x="27.945" y="22.38375" extent="1-16" drill="0.6"/>
+<wire x1="22.865" y1="22.38375" x2="27.94" y2="22.38375" width="0.4064" layer="16"/>
+<wire x1="27.94" y1="22.38375" x2="27.94" y2="22.5425" width="0.4064" layer="16"/>
+<wire x1="27.94" y1="22.5425" x2="27.945" y2="26.225" width="0.4064" layer="16"/>
+<via x="27.945" y="26.225" extent="1-16" drill="0.6"/>
 <contactref element="C11" pad="+"/>
-<wire x1="8.26" y1="30.559375" x2="8.26" y2="28.535" width="0.4064" layer="1"/>
+<wire x1="8.26" y1="30.32125" x2="8.26" y2="28.535" width="0.4064" layer="1"/>
 <contactref element="C7" pad="1"/>
 <contactref element="C9" pad="1"/>
@@
 <wire x1="26.065625" y1="26.151875" x2="26.04" y2="26.151875" width="0.4064" layer="1"/>
 <wire x1="26.04" y1="26.151875" x2="26.04" y2="26.19375" width="0.4064" layer="1"/>
+<wire x1="27.945" y1="30.32125" x2="27.945" y2="26.225" width="0.4064" layer="16"/>
 </signal>
 <signal name="N$9">
@@
 <wire x1="18.42" y1="26.499" x2="18.42" y2="28.36" width="0.4064" layer="1"/>
 <wire x1="18.42" y1="28.36" x2="20.6425" y2="28.36" width="0.4064" layer="1"/>
-<wire x1="18.205" y1="28.575" x2="18.42" y2="28.36" width="0.4064" layer="1"/>
 <wire x1="23.5" y1="27.01" x2="23.5" y2="28.0425" width="0.254" layer="1"/>
 <wire x1="23.5" y1="28.0425" x2="23.1825" y2="28.36" width="0.254" layer="1"/>
@@
 <wire x1="26.04" y1="37.465" x2="26.04" y2="37.885" width="0.4064" layer="1"/>
 <wire x1="10.9025" y1="33.655" x2="10.9025" y2="34.29" width="0.4064" layer="1"/>
-<wire x1="10.9025" y1="34.29" x2="10.9025" y2="38.4175" width="0.4064" layer="1"/>
+<wire x1="10.9025" y1="34.29" x2="10.9025" y2="37.455625" width="0.4064" layer="1"/>
+<wire x1="10.9025" y1="37.455625" x2="10.9025" y2="38.4175" width="0.4064" layer="1"/>
 <wire x1="10.9025" y1="38.4175" x2="10.53875" y2="38.4175" width="0.4064" layer="1"/>
 <wire x1="10.9025" y1="33.655" x2="10.9025" y2="31.90875" width="0.4064" layer="1"/>
@@
 <via x="15.88" y="22.225" extent="1-16" drill="0.6"/>
 <contactref element="C12" pad="+"/>
-<wire x1="10.9025" y1="38.4175" x2="10.9025" y2="39.0625" width="0.4064" layer="1"/>
-<wire x1="10.9025" y1="39.0625" x2="13.045" y2="41.205" width="0.4064" layer="1"/>
+<wire x1="13.069375" y1="37.455625" x2="10.9025" y2="37.455625" width="0.4064" layer="1"/>
 </signal>
 <signal name="N$1">
@@
 <contactref element="C13" pad="+"/>
 <wire x1="13.49875" y1="56.03875" x2="12.705" y2="55.245" width="0.4064" layer="1"/>
-<wire x1="12.705" y1="55.245" x2="12.705" y2="53.935" width="0.4064" layer="1"/>
+<wire x1="12.705" y1="55.245" x2="13.0225" y2="53.855625" width="0.4064" layer="1"/>
 <wire x1="10.53875" y1="54.2925" x2="12.3475" y2="54.2925" width="0.4064" layer="1"/>
-<wire x1="12.3475" y1="54.2925" x2="12.705" y2="53.935" width="0.4064" layer="1"/>
+<wire x1="12.3475" y1="54.2925" x2="13.0225" y2="53.855625" width="0.4064" layer="1"/>
 </signal>
 <signal name="N$2">
