File: thermostat_esp32_hw/thermostat_sensor_esp32.brd (EAGLE design)
At the start: 99.6 x 88 mm, 52 parts, among them IC2 ESP32-WROOM-32UE-N16, J1 TB-5.08-P-2P_BL, J2 TB-5.08-P-2P_BL, J3 TB-5.08-P-2P_BL, K1 G5LE-1_5VDC, K2 G5LE-1_5VDC, Q1 TLP185_SE_T, Q2 TLP185_SE_T

Commit message: different voltage regulator
Parts:
- removed PS1: LDI8119-3.3EN-DIO, AP2202K-3.3TRG1:SOT95P282X145-5N
- added IC1: TLV1117LV33DCYR, TLV1117LV33DCYR:SOT230P700X180-4N
- moved C10 7.30 mm to (17.4, 57.2)
- moved D2 7.30 mm to (19.8, 56.8)
- moved C11 7.30 mm to (23.9, 57.0)
- moved C12 7.30 mm to (11.7, 58.3)
- moved C3 7.30 mm to (25.9, 57.0)
- moved D1 7.30 mm to (22.3, 58.8)
- moved R1 7.30 mm to (22.3, 55.0)
- moved R4 0.48 mm to (3.40, 65.6)
- moved R5 0.48 mm to (3.43, 63.0)
- moved R18 0.32 mm to (3.30, 73.2)
Connections:
- net GND: now also IC1.1; no longer PS1.2
- net VCC3V3: now also IC1.2, IC1.4; no longer PS1.5
- net VCC5V: now also IC1.3; no longer PS1.1, PS1.3
Routing:
- net VCC5V: track 181.9 -> 195.3 mm, vias 4 -> 2
- net VCC3V3: track 203.5 -> 211.8 mm
- net GND: track 148.0 -> 153.0 mm, vias 6 -> 23
Other:
- board size 99.6 x 88 mm -> 96 x 88 mm

Commit message: minor pcb adjustments
Connections:
- net CLK: now also IC2.30; no longer IC2.33
- net DQ2: now also IC2.33; no longer IC2.30
Routing:
- net GND: track 153.0 -> 135.7 mm, vias 23 -> 27
- net VCC3V3: track 211.8 -> 200.6 mm, vias 5 -> 8
- net CLK: track 30.4 -> 33.8 mm, vias 0 -> 1
- net CS: track 30.6 -> 28.4 mm, vias 1 -> 2
- net DQ2: track 44.5 -> 42.8 mm
- net TXD0: track 54.9 -> 53.4 mm
- net RELAY1: track 34.3 -> 35.7 mm
- net VCC5V: track 195.3 -> 194.2 mm, vias 2 -> 3
- net RELAY2: track 56.9 -> 58.0 mm
- net RXD0: track 46.5 -> 47.6 mm
- net BOOT: track 42.9 -> 42.1 mm
- net EN: track 30.4 -> 31.0 mm

Commit message: fixes to fw and hw of thermostat
Parts:
- R11, R16: value 120 R -> 0 R
Changed lines of the file:
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@@
 <setting verticaltext="up"/>
 </settings>
-<grid distance="0.15875" unitdist="mm" unit="mm" style="dots" multiple="1" display="yes" altdistance="0.635" altunitdist="mm" altunit="mm"/>
+<grid distance="0.15875" unitdist="mm" unit="mm" style="dots" multiple="1" display="yes" altdistance="0.01" altunitdist="mm" altunit="mm"/>
 <layers>
 <layer number="1" name="Top" color="4" fill="1" visible="yes" active="yes"/>
@@
 <element name="R7" library="microbuilder" package="_0603" value="1k" x="63.97625" y="58.26125" smashed="yes"/>
 <element name="R10" library="microbuilder" package="_0603" value="10k" x="64.77" y="54.9275" smashed="yes" rot="R270"/>
-<element name="R11" library="microbuilder" package="_0603" value="120 R" x="62.865" y="54.9275" smashed="yes" rot="R90"/>
+<element name="R11" library="microbuilder" package="_0603" value="0 R" x="62.865" y="54.9275" smashed="yes" rot="R90"/>
 <element name="J2" library="TB-5.08-P-2P_BL" package="TB508P2PBL" value="TB-5.08-P-2P_BL" x="53.24475" y="5.49275" smashed="yes" rot="R180">
 <attribute name="TME_ELECTRONIC_COMPONENTS_PART_NUMBER" value="" x="53.24475" y="5.49275" size="1.778" layer="27" rot="R180" display="off"/>
@@
 <element name="R14" library="microbuilder" package="_0603" value="1k" x="83.21675" y="58.38825" smashed="yes"/>
 <element name="R15" library="microbuilder" package="_0603" value="10k" x="84.10575" y="55.02275" smashed="yes" rot="R270"/>
-<element name="R16" library="microbuilder" package="_0603" value="120 R" x="82.1055" y="55.02275" smashed="yes" rot="R90"/>
+<element name="R16" library="microbuilder" package="_0603" value="0 R" x="82.1055" y="55.02275" smashed="yes" rot="R90"/>
 <element name="J3" library="TB-5.08-P-2P_BL" package="TB508P2PBL" value="TB-5.08-P-2P_BL" x="80.54975" y="5.49275" smashed="yes" rot="R180">
 <attribute name="TME_ELECTRONIC_COMPONENTS_PART_NUMBER" value="" x="85.43925" y="21.30425" size="1.778" layer="27" rot="R180" display="off"/>
@@
 </signal>
 </signals>
-<errors>
-</errors>
 </board>
 </drawing>

Commit message: orp module added on thermostat base board
Parts:
- added U$21: ORP_PROBE, other:ORP_PROBE
Connections:
- net AC_N: now also U$1.P2; no longer U$1.P1
- net GND: now also U$21.GND
- net N$4: now also U$1.P1; no longer U$1.P2
- net RELAY1: now also U$21.SDA
- net RELAY2: now also U$21.SCL
- net VCC3V3: now also U$21.VCC3V3
- net VCC5V: now also U$21.VCC5V
Routing:
- net VCC3V3: track 200.6 -> 219.5 mm
- net RELAY1: track 35.7 -> 51.5 mm
- net RELAY2: track 58.0 -> 69.9 mm
- net AC_N: track 104.5 -> 93.7 mm
- net VCC5V: track 194.2 -> 202.8 mm
- net N$4: track 14.1 -> 8.25 mm
- net GND: vias 27 -> 25
Changed lines of the file:
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@@
 <setting verticaltext="up"/>
 </settings>
-<grid distance="0.15875" unitdist="mm" unit="mm" style="dots" multiple="1" display="yes" altdistance="0.01" altunitdist="mm" altunit="mm"/>
+<grid distance="0.15875" unitdist="mm" unit="mm" style="dots" multiple="1" display="yes" altdistance="0.15875" altunitdist="mm" altunit="mm"/>
 <layers>
 <layer number="1" name="Top" color="4" fill="1" visible="yes" active="yes"/>
@@
 <layer number="14" name="Route14" color="1" fill="6" visible="no" active="no"/>
 <layer number="15" name="Route15" color="4" fill="6" visible="no" active="no"/>
-<layer number="16" name="Bottom" color="1" fill="1" visible="no" active="yes"/>
+<layer number="16" name="Bottom" color="1" fill="1" visible="yes" active="yes"/>
 <layer number="17" name="Pads" color="2" fill="1" visible="yes" active="yes"/>
 <layer number="18" name="Vias" color="2" fill="1" visible="yes" active="yes"/>
@@
 <layer number="20" name="Dimension" color="15" fill="1" visible="yes" active="yes"/>
 <layer number="21" name="tPlace" color="14" fill="1" visible="yes" active="yes"/>
-<layer number="22" name="bPlace" color="11" fill="1" visible="no" active="yes"/>
+<layer number="22" name="bPlace" color="11" fill="1" visible="yes" active="yes"/>
 <layer number="23" name="tOrigins" color="15" fill="1" visible="yes" active="yes"/>
 <layer number="24" name="bOrigins" color="15" fill="1" visible="no" active="yes"/>
@@
 <wire x1="87.3125" y1="47.46625" x2="88.265" y2="46.51375" width="1.016" layer="46"/>
 <wire x1="88.265" y1="46.51375" x2="88.265" y2="39.21125" width="1.016" layer="46"/>
-<text x="9.8425" y="39.0525" size="1.778" layer="16" font="vector" ratio="20" rot="MR0">N</text>
+<text x="9.68375" y="28.09875" size="1.778" layer="16" font="vector" ratio="20" rot="MR0">N</text>
 <text x="16.35125" y="4.92125" size="1.778" layer="16" font="vector" ratio="20" rot="MR0">N</text>
 <text x="46.355" y="4.7625" size="1.778" layer="16" font="vector" ratio="20" rot="MR0">N</text>
@@
 <text x="87.15375" y="0.635" size="1.778" layer="16" font="vector" ratio="20" rot="MR0">L HEAT</text>
 <text x="63.8175" y="35.71875" size="1.778" layer="16" font="vector" ratio="20" rot="MR0">L</text>
+<text x="9.36625" y="41.275" size="1.778" layer="16" font="vector" ratio="20" rot="MR0">L</text>
 </plain>
 <attributes>
@@
 <attribute name="MANUFACTURER_PART_NUMBER" value="TLV1117LV33DCYR" x="33.49625" y="56.99125" size="1.778" layer="27" display="off"/>
 </element>
+<element name="U$21" library="other" package="ORP_PROBE" value="ORP_PROBE" x="56.8325" y="7.3025"/>
 </elements>
 <signals>
@@
 <via x="64.77" y="52.705" extent="1-16" drill="0.6"/>
 <via x="60.96" y="52.705" extent="1-16" drill="0.6"/>
-<via x="78.74" y="60.16625" extent="1-16" drill="0.6"/>
 <via x="84.1375" y="52.86375" extent="1-16" drill="0.6"/>
 <wire x1="49.89825" y1="29.11475" x2="52.07" y2="31.2865" width="1.016" layer="1"/>
@@
 <via x="75.72375" y="69.215" extent="1-16" drill="0.6"/>
 <via x="65.405" y="63.02375" extent="1-16" drill="0.6"/>
-<via x="84.61375" y="63.02375" extent="1-16" drill="0.6"/>
 <wire x1="75.565" y1="75.8825" x2="65.24625" y2="75.8825" width="0.4064" layer="16"/>
 <wire x1="65.24625" y1="75.8825" x2="64.92875" y2="76.2" width="0.4064" layer="16"/>
@@
 <via x="50.32375" y="83.97875" extent="1-16" drill="0.6"/>
 <via x="45.085" y="84.1375" extent="1-16" drill="0.6"/>
+<contactref element="U$21" pad="GND"/>
 </signal>
 <signal name="VCC5V">
@@
 <wire x1="10.00125" y1="51.435" x2="10.00125" y2="56.54675" width="1.016" layer="16"/>
 <wire x1="10.00125" y1="56.54675" x2="11.71575" y2="58.26125" width="1.016" layer="16"/>
+<contactref element="U$21" pad="VCC5V"/>
+<wire x1="88.9" y1="56.59875" x2="88.9" y2="59.53125" width="0.4064" layer="1"/>
+<wire x1="88.9" y1="59.53125" x2="88.5825" y2="59.84875" width="0.4064" layer="1"/>
+<wire x1="88.5825" y1="59.84875" x2="84.7725" y2="59.84875" width="0.4064" layer="1"/>
+<wire x1="84.7725" y1="59.84875" x2="84.455" y2="60.16625" width="0.4064" layer="1"/>
+<wire x1="84.455" y1="60.16625" x2="84.455" y2="61.1225" width="0.4064" layer="1"/>
+<wire x1="84.455" y1="61.1225" x2="84.4525" y2="61.1225" width="0.4064" layer="1"/>
 </signal>
 <signal name="EN">
@@
 </signal>
 <signal name="N$4">
-<contactref element="U$1" pad="P2"/>
+<contactref element="U$1" pad="P1"/>
 <contactref element="U$20" pad="P$2"/>
-<wire x1="11.39825" y1="29.11475" x2="3.175" y2="37.338" width="1.778" layer="16"/>
-<wire x1="3.175" y1="37.338" x2="3.175" y2="39.79925" width="1.778" layer="16"/>
+<wire x1="3.175" y1="39.79925" x2="11.33275" y2="39.79925" width="1.778" layer="16"/>
+<wire x1="11.33275" y1="39.79925" x2="11.39825" y2="39.86475" width="1.778" layer="16"/>
 </signal>
 <signal name="AC_N">
 <contactref element="J1" pad="2"/>
-<contactref element="U$1" pad="P1"/>
+<contactref element="U$1" pad="P2"/>
 <contactref element="J2" pad="2"/>
 <contactref element="J3" pad="2"/>
-<wire x1="18.31975" y1="5.49275" x2="18.31975" y2="2.54" width="1.778" layer="16"/>
+<wire x1="18.31975" y1="5.49275" x2="18.31975" y2="3.7818625" width="1.778" layer="16"/>
+<wire x1="18.31975" y1="3.7818625" x2="18.31975" y2="2.54" width="1.778" layer="16"/>
 <wire x1="18.31975" y1="2.54" x2="18.95475" y2="1.905" width="1.778" layer="16"/>
 <wire x1="18.95475" y1="1.905" x2="48.10125" y2="1.905" width="1.778" layer="16"/>
@@
 <wire x1="74.83475" y1="1.905" x2="75.46975" y2="2.54" width="1.778" layer="16"/>
 <wire x1="75.46975" y1="2.54" x2="75.46975" y2="5.49275" width="1.778" layer="16"/>
-<wire x1="18.31975" y1="5.49275" x2="18.31975" y2="32.94325" width="1.778" layer="16"/>
-<wire x1="18.31975" y1="32.94325" x2="11.39825" y2="39.86475" width="1.778" layer="16"/>
+<wire x1="18.31975" y1="5.49275" x2="18.31975" y2="22.19325" width="1.778" layer="16"/>
+<wire x1="18.31975" y1="22.19325" x2="11.39825" y2="29.11475" width="1.778" layer="16"/>
 </signal>
 <signal name="N$6">
@@
 <wire x1="69.469" y1="68.48475" x2="69.469" y2="67.21475" width="0.4064" layer="1"/>
 <wire x1="69.37375" y1="68.58" x2="69.37375" y2="72.54875" width="0.4064" layer="16"/>
+<contactref element="U$21" pad="SDA"/>
+<wire x1="79.3725" y1="61.1225" x2="79.3725" y2="66.89725" width="0.4064" layer="1"/>
+<wire x1="79.3725" y1="66.89725" x2="79.055" y2="67.21475" width="0.4064" layer="1"/>
+<wire x1="79.055" y1="67.21475" x2="69.469" y2="67.21475" width="0.4064" layer="1"/>
 </signal>
 <signal name="N$8">
@@
 <wire x1="39.13475" y1="76.5415" x2="49.1885" y2="76.5415" width="0.4064" layer="1"/>
 <wire x1="49.1885" y1="76.5415" x2="50.95875" y2="74.77125" width="0.4064" layer="1"/>
-<wire x1="70.64375" y1="73.025" x2="88.5825" y2="73.025" width="0.4064" layer="16"/>
+<wire x1="70.64375" y1="73.025" x2="76.8325" y2="73.025" width="0.4064" layer="16"/>
+<wire x1="76.835" y1="73.025" x2="88.5825" y2="73.025" width="0.4064" layer="16"/>
 <wire x1="88.5825" y1="73.025" x2="88.9" y2="72.7075" width="0.4064" layer="16"/>
 <wire x1="88.9" y1="72.7075" x2="88.9" y2="71.91375" width="0.4064" layer="16"/>
@@
 <wire x1="59.84875" y1="72.39" x2="57.4675" y2="74.77125" width="0.4064" layer="16"/>
 <wire x1="57.4675" y1="74.77125" x2="51.27625" y2="74.77125" width="0.4064" layer="16"/>
+<contactref element="U$21" pad="SCL"/>
+<wire x1="76.8325" y1="61.1225" x2="76.8325" y2="73.025" width="0.4064" layer="16"/>
+<wire x1="76.8325" y1="73.025" x2="76.835" y2="73.025" width="0.4064" layer="16"/>
 </signal>
 <signal name="N$13">
@@
 <wire x1="46.6725" y1="69.215" x2="46.6725" y2="73.66" width="0.8128" layer="16"/>
 <wire x1="46.6725" y1="73.66" x2="47.14875" y2="74.13625" width="0.8128" layer="16"/>
-<wire x1="41.11625" y1="58.80625" x2="41.11625" y2="61.75375" width="0.8128" layer="1"/>
-<wire x1="41.11625" y1="61.75375" x2="41.11625" y2="61.9125" width="0.8128" layer="1"/>
+<wire x1="41.11625" y1="58.80625" x2="41.11625" y2="62.32525" width="0.8128" layer="1"/>
 <wire x1="40.50525" y1="58.19525" x2="40.685" y2="58.375" width="0.4064" layer="1"/>
 <wire x1="40.685" y1="58.375" x2="41.11625" y2="58.80625" width="0.4064" layer="1"/>
@@
 <wire x1="46.355" y1="62.32525" x2="46.6725" y2="62.64275" width="0.8128" layer="1"/>
 <wire x1="46.6725" y1="62.64275" x2="46.6725" y2="69.215" width="0.8128" layer="1"/>
-<wire x1="41.11625" y1="61.9125" x2="41.11625" y2="62.32525" width="0.8128" layer="1"/>
+<contactref element="U$21" pad="VCC3V3"/>
+<wire x1="81.9125" y1="61.1225" x2="81.9125" y2="70.32375" width="0.4064" layer="1"/>
+<wire x1="81.9125" y1="70.32375" x2="85.852" y2="74.26325" width="0.4064" layer="1"/>
+<wire x1="85.852" y1="74.26325" x2="85.852" y2="78.4225" width="0.4064" layer="1"/>
 </signal>
 <signal name="N$19">
@@
 </signal>
 </signals>
+<errors>
+</errors>
 </board>
 </drawing>
